Commit message: Testing self collision avoidance

File: test/ur_description/urdf/ur10_robot.urdf (robot description, URDF)
Before this commit: robot ur5, 11 links, 10 joints
Links:
- link base: mass 0 -> 0.0
- link ee_link: mass 0 -> 0.0
- link forearm_link: mass 2.275 -> 3.87
- link shoulder_link: mass 3.7 -> 7.778
- link tool0: mass 0 -> 0.0
- link upper_arm_link: mass 8.393 -> 12.93
- link wrist_1_link: mass 1.219 -> 1.96
- link wrist_2_link: mass 1.219 -> 1.96
- link wrist_3_link: mass 0.1879 -> 0.202
Joints:
- joint ee_fixed_joint: origin xyz=0.0 0.0823 0.0 rpy=0.0 0.0 1.57079632679 -> xyz=0.0 0.0922 0.0 rpy=0.0 0.0 1.57079632679
- joint elbow_joint: origin xyz=0.0 -0.1197 0.425 rpy=0.0 0.0 0.0 -> xyz=0.0 -0.1719 0.612 rpy=0.0 0.0 0.0
- joint shoulder_lift_joint: limit lower=-6.28318530718 upper=6.28318530718 effort=150.0 velocity=3.15 -> lower=-6.28318530718 upper=6.28318530718 effort=330.0 velocity=2.16; origin xyz=0.0 0.13585 0.0 rpy=0.0 1.57079632679 0.0 -> xyz=0.0 0.220941 0.0 rpy=0.0 1.57079632679 0.0
- joint shoulder_pan_joint: limit lower=-6.28318530718 upper=6.28318530718 effort=150.0 velocity=3.15 -> lower=-6.28318530718 upper=6.28318530718 effort=330.0 velocity=2.16; origin xyz=0.0 0.0 0.089159 rpy=0.0 0.0 0.0 -> xyz=0.0 0.0 0.1273 rpy=0.0 0.0 0.0
- joint wrist_1_joint: limit lower=-6.28318530718 upper=6.28318530718 effort=28.0 velocity=3.2 -> lower=-6.28318530718 upper=6.28318530718 effort=54.0 velocity=3.2; origin xyz=0.0 0.0 0.39225 rpy=0.0 1.57079632679 0.0 -> xyz=0.0 0.0 0.5723 rpy=0.0 1.57079632679 0.0
- joint wrist_2_joint: limit lower=-6.28318530718 upper=6.28318530718 effort=28.0 velocity=3.2 -> lower=-6.28318530718 upper=6.28318530718 effort=54.0 velocity=3.2; origin xyz=0.0 0.093 0.0 rpy=0.0 0.0 0.0 -> xyz=0.0 0.1149 0.0 rpy=0.0 0.0 0.0
- joint wrist_3_joint: limit lower=-6.28318530718 upper=6.28318530718 effort=28.0 velocity=3.2 -> lower=-6.28318530718 upper=6.28318530718 effort=54.0 velocity=3.2; origin xyz=0.0 0.0 0.09465 rpy=0.0 0.0 0.0 -> xyz=0.0 0.0 0.1157 rpy=0.0 0.0 0.0
- joint wrist_3_link-tool0_fixed_joint: origin xyz=0 0.0823 0 rpy=-1.57079632679 0 0 -> xyz=0 0.0922 0 rpy=-1.57079632679 0 0
